File: pcb_matthieuT/RC_PCB_pro_v2.kicad_sch (KiCad schematic)
At the start: 14 parts

Commit message: Schematic and D real estate corrections
Parts:
- R1: value R_HC05_RX -> R_HC05_RX 470 kΩ
- R2: value R_HC05_GND -> R_HC05_GND 1 kΩ
- R_JS1: renamed from R_JS_right1; value R -> 47 kΩ
- R_button_left1, R_button_right1: value R -> 47 kΩ
- TM1637: footprint Connector_PinSocket_2.54mm:PinSocket_1x04_P2.54mm_Horizontal -> Connector_PinSocket_2.54mm:PinSocket_1x04_P2.54mm_Vertical
- renumbered JS_right1 to JS1
Connections:
- net GND: now also A2.29 (GND)
- net JS_H: now reaches A2.20 (A1)
- net JS_H: now also JS1.H2 (H)
- net Button_JS_L: no longer names the net of A2.6 (D3)
- net Button_JS_R renamed Button_JS
- net HCEnable: no longer names the net of HC05.6 (Pin_6)
- net HCEnable: no longer A2.16 (D13)
- net HCState: no longer names the net of HC05.1 (Pin_1)
- net HCState: no longer A2.15 (D12)
- net Left_H: no longer names the net of A2.25 (A6)
- net Left_V: no longer names the net of A2.23 (A4)
- net Right_H: no longer names the net of A2.21 (A2)
- net Right_H: no longer JS1.H2 (H)
- net Right_V renamed JS_V
Changed lines of the file:
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@@
+	)
+	(junction
+		(at 162.56 146.05)
+		(diameter 0)
+		(color 0 0 0 0)
 	)
 	(junction
@@
 	(wire
 		(pts
+			(xy 162.56 146.05) (xy 165.1 146.05)
+		)
+		(stroke
+			(width 0)
+			(type default)
+		)
+	)
+	(wire
+		(pts
 			(xy 162.56 146.05) (xy 162.56 154.94)
 		)
@@
 	(wire
 		(pts
-			(xy 167.64 52.07) (xy 167.64 38.1)
-		)
-		(stroke
-			(width 0)
-			(type default)
-		)
-	)
-	(wire
-		(pts
 			(xy 72.39 29.21) (xy 72.39 26.67)
 		)
@@
 	(wire
 		(pts
-			(xy 140.97 113.03) (xy 149.86 113.03)
-		)
-		(stroke
-			(width 0)
-			(type default)
-		)
-	)
-	(wire
-		(pts
 			(xy 72.39 36.83) (xy 86.36 36.83)
 		)
@@
 	(wire
 		(pts
-			(xy 137.16 135.89) (xy 149.86 135.89)
-		)
-		(stroke
-			(width 0)
-			(type default)
-		)
-	)
-	(wire
-		(pts
 			(xy 160.02 87.63) (xy 160.02 95.25)
 		)
@@
 	(wire
 		(pts
-			(xy 182.88 125.73) (xy 175.26 125.73)
-		)
-		(stroke
-			(width 0)
-			(type default)
-		)
-	)
-	(wire
-		(pts
 			(xy 167.64 90.17) (xy 167.64 95.25)
 		)
@@
 	(wire
 		(pts
-			(xy 154.94 40.64) (xy 154.94 38.1)
-		)
-		(stroke
-			(width 0)
-			(type default)
-		)
-	)
-	(wire
-		(pts
 			(xy 133.35 123.19) (xy 149.86 123.19)
 		)
@@
 	(wire
 		(pts
-			(xy 182.88 130.81) (xy 175.26 130.81)
-		)
-		(stroke
-			(width 0)
-			(type default)
-		)
-	)
-	(wire
-		(pts
 			(xy 44.45 66.04) (xy 44.45 35.56)
 		)
@@
 	(wire
 		(pts
-			(xy 138.43 138.43) (xy 149.86 138.43)
-		)
-		(stroke
-			(width 0)
-			(type default)
-		)
-	)
-	(wire
-		(pts
 			(xy 157.48 50.8) (xy 157.48 57.15)
 		)
@@
 	(wire
 		(pts
-			(xy 182.88 135.89) (xy 175.26 135.89)
-		)
-		(stroke
-			(width 0)
-			(type default)
-		)
-	)
-	(wire
-		(pts
 			(xy 87.63 166.37) (xy 90.17 166.37)
 		)
@@
 		(pts
 			(xy 157.48 38.1) (xy 157.48 50.8)
+		)
+		(stroke
+			(width 0)
+			(type default)
+		)
+	)
+	(wire
+		(pts
+			(xy 182.88 123.19) (xy 175.26 123.19)
 		)
 		(stroke
@@
 		)
 	)
-	(label "HCEnable"
-		(at 167.64 52.07 270)
+	(label "JS_H"
+		(at 182.88 123.19 0)
 		(effects
 			(font
 				(size 1.27 1.27)
 			)
-			(justify right bottom)
+			(justify left bottom)
 		)
 	)
@@
 		)
 	)
-	(label "HCState"
-		(at 154.94 40.64 270)
-		(effects
-			(font
-				(size 1.27 1.27)
-			)
-			(justify right bottom)
-		)
-	)
 	(label "TX"
 		(at 160.02 53.34 0)
@@
 		)
 	)
-	(label "Button_JS_L"
-		(at 140.97 113.03 180)
-		(effects
-			(font
-				(size 1.27 1.27)
-			)
-			(justify right bottom)
-		)
-	)
 	(label "TX"
 		(at 132.08 128.27 180)
@@
 		)
 	)
-	(label "HCState"
-		(at 137.16 135.89 180)
-		(effects
-			(font
-				(size 1.27 1.27)
-			)
-			(justify right bottom)
-		)
-	)
-	(label "Right_V"
+	(label "JS_V"
 		(at 236.22 102.87 180)
 		(effects
@@
 		)
 	)
-	(label "Button_JS_R"
+	(label "Button_JS"
 		(at 140.97 110.49 180)
 		(fields_autoplaced yes)
@@
 		)
 	)
-	(label "Left_H"
-		(at 182.88 135.89 0)
-		(effects
-			(font
-				(size 1.27 1.27)
-			)
-			(justify left bottom)
-		)
-	)
-	(label "Left_V"
-		(at 182.88 130.81 0)
-		(effects
-			(font
-				(size 1.27 1.27)
-			)
-			(justify left bottom)
-		)
-	)
-	(label "HCEnable"
-		(at 138.43 138.43 180)
-		(effects
-			(font
-				(size 1.27 1.27)
-			)
-			(justify right bottom)
-		)
-	)
 	(label "DIO"
 		(at 116.84 78.74 0)
@@
 		)
 	)
-	(label "Button_JS_R"
+	(label "Button_JS"
 		(at 215.9 125.73 0)
 		(effects
@@
 		)
 	)
-	(label "Right_V"
+	(label "JS_V"
 		(at 182.88 120.65 0)
-		(effects
-			(font
-				(size 1.27 1.27)
-			)
-			(justify left bottom)
-		)
-	)
-	(label "Right_H"
-		(at 182.88 125.73 0)
 		(effects
 			(font
@@
 		)
 	)
-	(label "Right_H"
+	(label "JS_H"
 		(at 236.22 113.03 180)
 		(effects
@@
 			)
 		)
-		(property "Value" "R"
+		(property "Value" "47 kΩ"
 			(at 236.22 31.7499 0)
 			(effects
@@
 			)
 		)
-		(property "Value" "R"
+		(property "Value" "47 kΩ"
 			(at 74.93 34.2899 0)
 			(effects
@@
 			)
 		)
-		(property "Value" "R_HC05_GND"
+		(property "Value" "R_HC05_GND 1 kΩ"
 			(at 146.05 46.99 90)
 			(effects
@@
 		(dnp no)
 		(fields_autoplaced yes)
-		(property "Reference" "JS_right1"
+		(property "Reference" "JS1"
 			(at 266.7 115.5699 0)
 			(effects
@@
 			(project ""
 				(path "/215bf3d6-76c1-4027-ae44-8a7d4ae3c8e5"
-					(reference "JS_right1")
+					(reference "JS1")
 					(unit 1)
 				)
@@
 		(dnp no)
 		(fields_autoplaced yes)
-		(property "Reference" "R_JS_right1"
+		(property "Reference" "R_JS1"
 			(at 233.68 132.0799 0)
 			(effects
@@
 			)
 		)
-		(property "Value" "R"
+		(property "Value" "47 kΩ"
 			(at 233.68 134.6199 0)
 			(effects
@@
 			(project "RC_PCB_pro"
 				(path "/215bf3d6-76c1-4027-ae44-8a7d4ae3c8e5"
-					(reference "R_JS_right1")
+					(reference "R_JS1")
 					(unit 1)
 				)
@@
 			)
 		)
-		(property "Value" "R_HC05_RX"
+		(property "Value" "R_HC05_RX 470 kΩ"
 			(at 160.02 60.9599 0)
 			(effects
@@
 			)
 		)
-		(property "Footprint" "Connector_PinSocket_2.54mm:PinSocket_1x04_P2.54mm_Horizontal"
+		(property "Footprint" "Connector_PinSocket_2.54mm:PinSocket_1x04_P2.54mm_Vertical"
 			(at 102.87 81.28 0)
 			(effects
